File: test/test.kicad_sch (KiCad schematic)
At the start: 68 parts, among them Y1 NI

Commit message: wip
Parts:
- removed L2: ~, symbol Logos:Rancune
- BAT1: symbol Generiques:BAT -> Generics:BAT
- BAT2: symbol Generiques:BAT_Multicell -> Generics:BAT_Multicell
- BR1: value ~ -> (none); symbol Generiques:BR -> Generics:BR
- C1: symbol Generiques:C -> Generics:C
- C2: symbol Generiques:C_Polarized -> Generics:C_Polarized
- C3: symbol Generiques:C_Polarized_alt -> Generics:C_Polarized_alt
- C4: symbol Generiques:C_alt -> Generics:C_alt
- C5: symbol Generiques_small:C_ -> Generics_small:C_
- C6: symbol Generiques_small:C_alt_ -> Generics_small:C_alt_
- C7: symbol Generiques_small:C_Polarized_ -> Generics_small:C_Polarized_
- C8: symbol Generiques_small:C_Polarized_alt_ -> Generics_small:C_Polarized_alt_
- D1: symbol Generiques:D_Zener -> Generics:D_Zener
- D10: value ~ -> (none); symbol Generiques:D_Schottky -> Generics:D_Schottky
- D11: value ~ -> (none); symbol Generiques:D -> Generics:D
- D13: value ~ -> (none); symbol Generiques:D_TVS_bidir -> Generics:D_TVS_bidir
- D2: value ~ -> (none); symbol Generiques:DIAC -> Generics:DIAC
- D3: value ~ -> (none); symbol Generiques:D_LED -> Generics:D_LED
- D4: value ~ -> (none); symbol Generiques:D_LED_blue -> Generics:D_LED_blue
- D5: value ~ -> (none); symbol Generiques:D_LED_green -> Generics:D_LED_green
- D6: value ~ -> (none); symbol Generiques:D_LED_red -> Generics:D_LED_red
- D7: value ~ -> (none); symbol Generiques:D_LED_yellow -> Generics:D_LED_yellow
- D8: value ~ -> (none); symbol Generiques:D_Photo -> Generics:D_Photo
- D9: value ~ -> (none); symbol Generiques:D_TVS -> Generics:D_TVS
- F1: symbol Generiques:F -> Generics:F
- FB1: symbol Generiques:FB -> Generics:FB
- J1: value ~ -> (none); symbol Generiques:J_Connector_1x2 -> Generics:J_Connector_1x2
- J10, Logo1, Logo2, Logo3, MH1, SB1, SB2, TP1: value ~ -> (none)
- J2: value ~ -> (none); symbol Generiques:J_Connector_1x3 -> Generics:J_Connector_1x3
- J3: value ~ -> (none); symbol Generiques:J_Connector_1x4 -> Generics:J_Connector_1x4
- J4: value ~ -> (none); symbol Generiques:J_Connector_1x5 -> Generics:J_Connector_1x5
- J5, J6: value ~ -> (none); symbol Generiques:J_Connector_1x6 -> Generics:J_Connector_1x6
- J7: value ~ -> (none); symbol Generiques:J_Connector_1x7 -> Generics:J_Connector_1x7
- J8: value ~ -> (none); symbol Generiques:J_Connector_1x8 -> Generics:J_Connector_1x8
- J9: value ~ -> (none); symbol Generiques:J_RJ45_w_Leds -> Generics:J_RJ45_w_Leds
- L1: symbol Generiques:L -> Generics:L
- OP1: value ~ -> (none); symbol Generiques:OP -> Generics:OP
- Q1: value ~ -> (none); symbol Generiques:Q_BJT_NPN -> Generics:Q_BJT_NPN
- Q2: value ~ -> (none); symbol Generiques:Q_MOSFET_N -> Generics:Q_MOSFET_N
- Q3: value ~ -> (none); symbol Generiques:Q_BJT_PNP -> Generics:Q_BJT_PNP
- Q4: value ~ -> (none); symbol Generiques:Q_MOSFET_P -> Generics:Q_MOSFET_P
- R1: symbol Generiques:R -> Generics:R
- R2: symbol Generiques:R_alt -> Generics:R_alt
- R3: symbol Generiques_small:R_ -> Generics_small:R_
- R4: symbol Generiques_small:R_alt_ -> Generics_small:R_alt_
- SW1: value ~ -> (none); symbol Generiques:SW_PushButton -> Generics:SW_PushButton
- SW2: value ~ -> (none); symbol Generiques:SW_PushButton_45deg -> Generics:SW_PushButton_45deg
- SW3: value ~ -> (none); symbol Generiques:SW_PushButton_Open -> Generics:SW_PushButton_Open
- SW4: value ~ -> (none); symbol Generiques:SW_Switch_DPST -> Generics:SW_Switch_DPST
- SW5: value ~ -> (none); symbol Generiques:SW_Switch_SPDT -> Generics:SW_Switch_SPDT
- SW6: value ~ -> (none); symbol Generiques:SW_Switch_SPST -> Generics:SW_Switch_SPST
- T1: value ~ -> (none); symbol Generiques:T_CT_Iron -> Generics:T_CT_Iron
- T2: value ~ -> (none); symbol Generiques:T_Dual_Iron -> Generics:T_Dual_Iron
- T3: value ~ -> (none); symbol Generiques:T_Simple_Air -> Generics:T_Simple_Air
- T4: value ~ -> (none); symbol Generiques:T_Simple_Ferrite -> Generics:T_Simple_Ferrite
- T5: value ~ -> (none); symbol Generiques:T_Simple_Iron -> Generics:T_Simple_Iron
- U1: value ~ -> (none); symbol Generiques:U_LDO_Fixed -> Generics:U_LDO_Fixed
- U2: value ~ -> (none); symbol Generiques:U_OPAMP -> Generics:U_OPAMP
- Y1: symbol Generiques:Y -> Generics:Y
