File: test/test_symbols/test.kicad_sch (KiCad schematic)
At the start: 67 parts, among them Y1 NI

Commit message: Logos integration
Parts:
- removed Logo2: (no value), symbol Logos:Logo_RoHS
- removed Logo3: (no value), symbol Logos:Logo_CE
- removed Logo4: (no value), symbol Logos:Logo_ISO_7010_W017
- added Logo2: ~, symbol Logos:Logo_CE
- added Logo3: ~, symbol Logos:Logo_RoHS
- added Logo4: ~, symbol Logos:Logo_ESD
- added Logo5: ~, symbol Logos:Logo_ISO_7010_W017
- BR1, D10, D11, D13, D2, D3, D4, D5, D6, D7, D8, D9, J1, J10, J2, J3, J4, J5, J6, J7, J8, J9, Logo1, MH1, OP1, Q1, Q2, Q3, Q4, SB1, SB2, SW1, SW2, SW3, SW4, SW5, SW6, T1, T2, T3, T4, T5, TP1, U1, U2: value (none) -> ~
